File: multivib.kicad_pcb (KiCad board)
At the start: 2 copper layers, 16 parts, among them J1 KLS2-301-5.00-02P-2S, J2 KLS2-301-5.00-02P-2S, J3 KLS2-301-5.00-02P-2S, Q1 BC817, Q2 BC817, Q3 2N7002

Commit message: плата
Parts:
- added H1: MountingHole, MountingHole:MountingHole_2.1mm, F.Cu at (109.2, 111.1)
- added H2: MountingHole, MountingHole:MountingHole_2.1mm, F.Cu at (132.1, 111.1)
- added H3: MountingHole, MountingHole:MountingHole_2.1mm, F.Cu at (132.1, 89.5)
- added H4: MountingHole, MountingHole:MountingHole_2.1mm, F.Cu at (109.2, 89.5)
- moved J2 8.25 mm to (123.1, 92.5)
- moved C3 7.01 mm to (113.0, 93.3)
- moved C4 7.01 mm to (113.0, 95.9)
- moved R5 4.45 mm to (128.3, 96.5)
- moved D1 4.02 mm to (131.4, 95.2), turned to -90 degrees
- moved Q3 3.70 mm to (128.3, 93.3)
Other:
- board outline added: 27.9 x 26.7 mm

Commit message: работа с разводкой
Parts:
- H1, H2, H3, H4: footprint MountingHole:MountingHole_2.1mm -> MountingHole:MountingHole_2.2mm_M2_DIN965
- moved J3 5.15 mm to (130.8, 105.4), turned to 90 degrees
- moved H4 2.28 mm to (107.0, 89.0)
- moved H1 2.22 mm to (107.0, 111.0)
- moved H3 1.99 mm to (134.0, 89.0)
- moved H2 1.92 mm to (134.0, 111.0)
- moved Q3 1.27 mm to (128.2, 92.1)
- turned Q1 to 180 degrees
Connections:
- J2 pad 1: Net-(C3-Pad1) -> GND
- J2 pad 2: GND -> Net-(C3-Pad1)
- J3 pad 1: /out2 -> GND
- J3 pad 2: GND -> /out2
Routing:
- net Net-(C3-Pad1): track 0.00 -> 25.0 mm
- net /out2: track 0.00 -> 23.1 mm, vias 0 -> 1
- net /out1: track 0.00 -> 12.8 mm
- net GND: track 0.00 -> 10.6 mm, vias 0 -> 5
- net Net-(C2-Pad2): track 0.00 -> 10.0 mm, vias 0 -> 2
- net Net-(C1-Pad1): track 0.00 -> 7.34 mm
- net Net-(D1-Pad1): track 0.00 -> 5.84 mm
- net Net-(D1-Pad2): track 0.00 -> 2.31 mm
- added copper zone on B.Cu, net GND
- added copper zone on F.Cu, net GND
Other:
- board size 27.9 x 26.7 mm -> 32.5 x 27.5 mm
- board text added: "+"
- board text added: "-"
- board text added: "OUT1"
- board text added: "OUT2"
- board text added: "PWR"
