File: multivib.kicad_sch (KiCad schematic)
At the start: 16 parts, among them J1 KLS2-301-5.00-02P-2S, J2 KLS2-301-5.00-02P-2S, J3 KLS2-301-5.00-02P-2S, Q1 BC817, Q2 BC817, Q3 2N7002

Commit message: работа с разводкой
Parts:
- added H1, H2, H3, H4: MountingHole, MountingHole:MountingHole_2.2mm_M2_DIN965, symbol Mechanical:MountingHole
Connections:
- net GND: now also J2.1, J3.1; no longer J2.2, J3.2
- net out2: now also J3.2; no longer J3.1
- net at C3.1, C4.1, R1.1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: now also J2.2; no longer J2.1
Other:
- moved on the sheet: J2
Changed lines of the file:
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@@
     (effects (font (size 1.27 1.27)) (justify left bottom))
   )
-  (symbol (lib_id "MAS_Connectors:KLS2-301-5.00-02P-2S") (at 209.55 109.22 0) (unit 1)
-    (in_bom yes) (on_board yes)
-    (property "Reference" "J3" (id 0) (at 213.36 107.95 0))
-    (property "Value" "KLS2-301-5.00-02P-2S" (id 1) (at 224.79 110.49 0))
-    (property "Footprint" "MAS_Package_nostd:KLS2-301-5.00-02P-2S" (id 2) (at 198.12 115.57 0)
-      (effects (font (size 1.27 1.27) italic) (justify left) hide)
-    )
-    (property "Datasheet" "https://static.chipdip.ru/lib/507/DOC001507148.pdf" (id 3) (at 208.28 44.45 0)
+  (symbol (lib_id "MAS_Connectors:KLS2-301-5.00-02P-2S") (at 209.55 109.22 0) (mirror x) (unit 1)
+    (in_bom yes) (on_board yes)
+    (property "Reference" "J3" (id 0) (at 213.36 110.49 0))
+    (property "Value" "KLS2-301-5.00-02P-2S" (id 1) (at 224.79 107.95 0))
+    (property "Footprint" "MAS_Package_nostd:KLS2-301-5.00-02P-2S" (id 2) (at 198.12 102.87 0)
+      (effects (font (size 1.27 1.27) italic) (justify left) hide)
+    )
+    (property "Datasheet" "https://static.chipdip.ru/lib/507/DOC001507148.pdf" (id 3) (at 208.28 173.99 0)
       (effects (font (size 1.27 1.27)) hide)
     )
@@
     (pin "1")
     (pin "2")
+  )
+  (symbol (lib_id "Mechanical:MountingHole") (at 186.69 128.27 0) (unit 1)
+    (in_bom yes) (on_board yes) (fields_autoplaced)
+    (property "Reference" "H2" (id 0) (at 189.23 126.9999 0)
+      (effects (font (size 1.27 1.27)) (justify left))
+    )
+    (property "Value" "MountingHole" (id 1) (at 189.23 129.5399 0)
+      (effects (font (size 1.27 1.27)) (justify left))
+    )
+    (property "Footprint" "MountingHole:MountingHole_2.2mm_M2_DIN965" (id 2) (at 186.69 128.27 0)
+      (effects (font (size 1.27 1.27)) hide)
+    )
+    (property "Datasheet" "~" (id 3) (at 186.69 128.27 0)
+      (effects (font (size 1.27 1.27)) hide)
+    )
   )
   (symbol (lib_id "Device:LED_Small") (at 184.15 93.98 90) (unit 1)
@@
     (pin "2")
   )
-  (symbol (lib_id "MAS_Connectors:KLS2-301-5.00-02P-2S") (at 82.55 102.87 0) (mirror y) (unit 1)
-    (in_bom yes) (on_board yes)
-    (property "Reference" "J2" (id 0) (at 78.74 101.6 0))
-    (property "Value" "KLS2-301-5.00-02P-2S" (id 1) (at 67.31 104.14 0))
-    (property "Footprint" "MAS_Package_nostd:KLS2-301-5.00-02P-2S" (id 2) (at 93.98 109.22 0)
-      (effects (font (size 1.27 1.27) italic) (justify left) hide)
-    )
-    (property "Datasheet" "https://static.chipdip.ru/lib/507/DOC001507148.pdf" (id 3) (at 83.82 38.1 0)
+  (symbol (lib_id "MAS_Connectors:KLS2-301-5.00-02P-2S") (at 82.55 102.87 180) (unit 1)
+    (in_bom yes) (on_board yes)
+    (property "Reference" "J2" (id 0) (at 78.74 104.14 0))
+    (property "Value" "KLS2-301-5.00-02P-2S" (id 1) (at 67.31 101.6 0))
+    (property "Footprint" "MAS_Package_nostd:KLS2-301-5.00-02P-2S" (id 2) (at 93.98 96.52 0)
+      (effects (font (size 1.27 1.27) italic) (justify left) hide)
+    )
+    (property "Datasheet" "https://static.chipdip.ru/lib/507/DOC001507148.pdf" (id 3) (at 83.82 167.64 0)
       (effects (font (size 1.27 1.27)) hide)
     )
@@
     (pin "3")
   )
+  (symbol (lib_id "Mechanical:MountingHole") (at 186.69 133.35 0) (unit 1)
+    (in_bom yes) (on_board yes) (fields_autoplaced)
+    (property "Reference" "H3" (id 0) (at 189.23 132.0799 0)
+      (effects (font (size 1.27 1.27)) (justify left))
+    )
+    (property "Value" "MountingHole" (id 1) (at 189.23 134.6199 0)
+      (effects (font (size 1.27 1.27)) (justify left))
+    )
+    (property "Footprint" "MountingHole:MountingHole_2.2mm_M2_DIN965" (id 2) (at 186.69 133.35 0)
+      (effects (font (size 1.27 1.27)) hide)
+    )
+    (property "Datasheet" "~" (id 3) (at 186.69 133.35 0)
+      (effects (font (size 1.27 1.27)) hide)
+    )
+  )
   (symbol (lib_id "MAS_Connectors:KLS2-301-5.00-02P-2S") (at 209.55 96.52 0) (unit 1)
     (in_bom yes) (on_board yes)
@@
     (pin "2")
   )
+  (symbol (lib_id "Mechanical:MountingHole") (at 186.69 123.19 0) (unit 1)
+    (in_bom yes) (on_board yes) (fields_autoplaced)
+    (property "Reference" "H1" (id 0) (at 189.23 121.9199 0)
+      (effects (font (size 1.27 1.27)) (justify left))
+    )
+    (property "Value" "MountingHole" (id 1) (at 189.23 124.4599 0)
+      (effects (font (size 1.27 1.27)) (justify left))
+    )
+    (property "Footprint" "MountingHole:MountingHole_2.2mm_M2_DIN965" (id 2) (at 186.69 123.19 0)
+      (effects (font (size 1.27 1.27)) hide)
+    )
+    (property "Datasheet" "~" (id 3) (at 186.69 123.19 0)
+      (effects (font (size 1.27 1.27)) hide)
+    )
+  )
   (symbol (lib_id "power:GND") (at 204.47 100.33 0) (unit 1)
     (in_bom yes) (on_board yes)
@@
     (pin "2")
   )
+  (symbol (lib_id "Mechanical:MountingHole") (at 186.69 138.43 0) (unit 1)
+    (in_bom yes) (on_board yes) (fields_autoplaced)
+    (property "Reference" "H4" (id 0) (at 189.23 137.1599 0)
+      (effects (font (size 1.27 1.27)) (justify left))
+    )
+    (property "Value" "MountingHole" (id 1) (at 189.23 139.6999 0)
+      (effects (font (size 1.27 1.27)) (justify left))
+    )
+    (property "Footprint" "MountingHole:MountingHole_2.2mm_M2_DIN965" (id 2) (at 186.69 138.43 0)
+      (effects (font (size 1.27 1.27)) hide)
+    )
+    (property "Datasheet" "~" (id 3) (at 186.69 138.43 0)
+      (effects (font (size 1.27 1.27)) hide)
+    )
+  )
   (symbol (lib_id "Device:R") (at 168.91 95.25 0) (unit 1)
     (in_bom yes) (on_board yes) (fields_autoplaced)
@@
       (reference "D1") (unit 1) (value "LED_Green") (footprint "LED_SMD:LED_0805_2012Metric")
     )
+    (path "/d8c0b89e-45fc-4c20-b824-badbed9aa764"
+      (reference "H1") (unit 1) (value "MountingHole") (footprint "MountingHole:MountingHole_2.2mm_M2_DIN965")
+    )
+    (path "/38982b0a-458e-40f6-9c9e-3ae02df83c97"
+      (reference "H2") (unit 1) (value "MountingHole") (footprint "MountingHole:MountingHole_2.2mm_M2_DIN965")
+    )
+    (path "/787a378d-ecce-4112-af45-52cf13207811"
+      (reference "H3") (unit 1) (value "MountingHole") (footprint "MountingHole:MountingHole_2.2mm_M2_DIN965")
+    )
+    (path "/dbe4f657-a017-4d41-9ec1-b14b8c6efa6b"
+      (reference "H4") (unit 1) (value "MountingHole") (footprint "MountingHole:MountingHole_2.2mm_M2_DIN965")
+    )
     (path "/7eb8d7f4-6d58-4e3b-a9ab-e8adbf54e369"
