File: hardware/multivib.kicad_pcb (KiCad board)
At the start: 2 copper layers, 32.5 x 27.5 mm, 20 parts, among them J1 KLS2-301-5.00-02P-2S, J2 KLS2-301-5.00-02P-2S, J3 KLS2-301-5.00-02P-2S, Q1 BC817, Q2 BC817, Q3 2N7002

Commit message: почти готово
Routing:
- net /out2: track 23.1 -> 22.2 mm
- net /out1: track 12.8 -> 12.1 mm
- net GND: vias 5 -> 35
Changed lines of the file:
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@@
     )
     (pad_to_mask_clearance 0)
-    (aux_axis_origin 104.68 113.665)
-    (grid_origin 104.68 113.665)
+    (aux_axis_origin 104.18 113.665)
+    (grid_origin 104.18 113.665)
     (pcbplotparams
       (layerselection 0x00010fc_ffffffff)
@@
     (pad "" np_thru_hole circle (at 0 0) (size 2.2 2.2) (drill 2.2) (layers *.Cu *.Mask))
   )
-  (gr_line (start 103.48 113.665) (end 105.88 113.665) (layer "Dwgs.User") (width 0.1))
-  (gr_line (start 104.68 112.665) (end 104.68 114.865) (layer "Dwgs.User") (width 0.1))
+  (gr_line (start 104.18 112.395) (end 104.18 114.935) (layer "Dwgs.User") (width 0.1))
+  (gr_line (start 105.45 113.665) (end 102.91 113.665) (layer "Dwgs.User") (width 0.1))
   (gr_line (start 107.18 113.665) (end 133.68 113.665) (layer "Edge.Cuts") (width 0.05))
   (gr_arc (start 107.18 113.665) (mid 105.05868 112.78632) (end 104.18 110.665) (layer "Edge.Cuts") (width 0.05))
@@
   (segment (start 119.06 101.825) (end 119.06 102.87) (width 0.25) (layer "F.Cu") (net 1))
   (segment (start 122.2525 104.5675) (end 122.2525 105.095) (width 0.25) (layer "F.Cu") (net 1))
-  (segment (start 119.38 100.695) (end 119.38 101.505) (width 0.25) (layer "F.Cu") (net 1))
   (segment (start 119.06 102.87) (end 119.06 103.915) (width 0.25) (layer "F.Cu") (net 1))
   (segment (start 119.38 101.505) (end 119.06 101.825) (width 0.25) (layer "F.Cu") (net 1))
+  (segment (start 119.38 100.695) (end 119.38 101.505) (width 0.25) (layer "F.Cu") (net 1))
   (segment (start 121.952 104.267) (end 122.2525 104.5675) (width 0.25) (layer "F.Cu") (net 1))
   (segment (start 119.06 103.915) (end 119.412 104.267) (width 0.25) (layer "F.Cu") (net 1))
-  (segment (start 117.1725 103.9915) (end 117.1725 106.045) (width 0.25) (layer "F.Cu") (net 2))
+  (segment (start 117.16 106.0325) (end 117.1725 106.045) (width 0.25) (layer "F.Cu") (net 2))
   (segment (start 114.602 100.457) (end 110.338 100.457) (width 0.25) (layer "F.Cu") (net 2))
   (segment (start 110.338 100.457) (end 110.3275 100.4675) (width 0.25) (layer "F.Cu") (net 2))
   (segment (start 114.84 100.695) (end 114.602 100.457) (width 0.25) (layer "F.Cu") (net 2))
-  (segment (start 117.16 103.979) (end 117.1725 103.9915) (width 0.25) (layer "F.Cu") (net 2))
-  (segment (start 116.57 100.965) (end 116.84 100.695) (width 0.25) (layer "F.Cu") (net 2))
-  (segment (start 117.16 101.761) (end 117.16 102.87) (width 0.25) (layer "F.Cu") (net 2))
-  (segment (start 116.84 101.441) (end 117.16 101.761) (width 0.25) (layer "F.Cu") (net 2))
-  (segment (start 117.16 102.87) (end 117.16 103.979) (width 0.25) (layer "F.Cu") (net 2))
+  (segment (start 117.16 101.88) (end 116.84 101.56) (width 0.25) (layer "F.Cu") (net 2))
+  (segment (start 116.84 101.56) (end 116.84 100.695) (width 0.25) (layer "F.Cu") (net 2))
+  (segment (start 117.16 102.87) (end 117.16 106.0325) (width 0.25) (layer "F.Cu") (net 2))
+  (segment (start 117.16 102.87) (end 117.16 101.88) (width 0.25) (layer "F.Cu") (net 2))
   (segment (start 116.84 100.695) (end 114.84 100.695) (width 0.25) (layer "F.Cu") (net 2))
-  (segment (start 117.38 102.65) (end 117.16 102.87) (width 0.25) (layer "F.Cu") (net 2))
-  (segment (start 116.84 100.695) (end 116.84 101.441) (width 0.25) (layer "F.Cu") (net 2))
-  (segment (start 121.92 101.441) (end 122.24 101.761) (width 0.25) (layer "F.Cu") (net 3))
-  (segment (start 121.92 100.695) (end 121.92 101.441) (width 0.25) (layer "F.Cu") (net 3))
+  (segment (start 121.92 101.56) (end 122.24 101.88) (width 0.25) (layer "F.Cu") (net 3))
   (segment (start 120.428 107.061) (end 119.1135 107.061) (width 0.25) (layer "F.Cu") (net 3))
-  (segment (start 122.24 101.761) (end 122.24 102.87) (width 0.25) (layer "F.Cu") (net 3))
-  (segment (start 122.46 102.65) (end 122.24 102.87) (width 0.25) (layer "F.Cu") (net 3))
+  (segment (start 121.92 100.695) (end 121.92 101.56) (width 0.25) (layer "F.Cu") (net 3))
   (segment (start 120.428 102.87) (end 122.24 102.87) (width 0.25) (layer "F.Cu") (net 3))
+  (segment (start 122.24 101.88) (end 122.24 102.87) (width 0.25) (layer "F.Cu") (net 3))
   (segment (start 119.1135 107.061) (end 119.0475 106.995) (width 0.25) (layer "F.Cu") (net 3))
   (via (at 120.428 102.87) (size 0.8) (drill 0.4) (layers "F.Cu" "B.Cu") (net 3))
@@
   (segment (start 110.395 93.345) (end 110.429 93.311) (width 0.25) (layer "F.Cu") (net 4))
   (segment (start 119.0475 105.095) (end 120.3525 105.095) (width 0.25) (layer "F.Cu") (net 4))
-  (via (at 133.89 93.345) (size 0.8) (drill 0.4) (layers "F.Cu" "B.Cu") (free) (net 4))
+  (via (at 114.34 111.125) (size 0.8) (drill 0.4) (layers "F.Cu" "B.Cu") (free) (net 4))
+  (via (at 116.88 95.885) (size 0.8) (drill 0.4) (layers "F.Cu" "B.Cu") (free) (net 4))
+  (via (at 132.12 108.585) (size 0.8) (drill 0.4) (layers "F.Cu" "B.Cu") (free) (net 4))
+  (via (at 124.5 111.125) (size 0.8) (drill 0.4) (layers "F.Cu" "B.Cu") (free) (net 4))
+  (via (at 119.42 95.885) (size 0.8) (drill 0.4) (layers "F.Cu" "B.Cu") (free) (net 4))
+  (via (at 114.34 108.585) (size 0.8) (drill 0.4) (layers "F.Cu" "B.Cu") (free) (net 4))
+  (via (at 124.5 95.885) (size 0.8) (drill 0.4) (layers "F.Cu" "B.Cu") (free) (net 4))
+  (via (at 111.8 90.805) (size 0.8) (drill 0.4) (layers "F.Cu" "B.Cu") (free) (net 4))
+  (via (at 114.34 88.265) (size 0.8) (drill 0.4) (layers "F.Cu" "B.Cu") (free) (net 4))
+  (via (at 114.34 106.045) (size 0.8) (drill 0.4) (layers "F.Cu" "B.Cu") (free) (net 4))
+  (via (at 109.26 90.805) (size 0.8) (drill 0.4) (layers "F.Cu" "B.Cu") (free) (net 4))
+  (via (at 119.42 111.125) (size 0.8) (drill 0.4) (layers "F.Cu" "B.Cu") (free) (net 4))
+  (via (at 124.5 108.585) (size 0.8) (drill 0.4) (layers "F.Cu" "B.Cu") (free) (net 4))
   (via (at 110.395 95.885) (size 0.8) (drill 0.4) (layers "F.Cu" "B.Cu") (net 4))
+  (via (at 109.26 108.585) (size 0.8) (drill 0.4) (layers "F.Cu" "B.Cu") (free) (net 4))
+  (via (at 129.58 111.125) (size 0.8) (drill 0.4) (layers "F.Cu" "B.Cu") (free) (net 4))
   (via (at 122.2568 108.4326) (size 0.8) (drill 0.4) (layers "F.Cu" "B.Cu") (net 4))
+  (via (at 129.58 88.265) (size 0.8) (drill 0.4) (layers "F.Cu" "B.Cu") (free) (net 4))
+  (via (at 134.66 95.885) (size 0.8) (drill 0.4) (layers "F.Cu" "B.Cu") (free) (net 4))
+  (via (at 114.34 103.505) (size 0.8) (drill 0.4) (layers "F.Cu" "B.Cu") (free) (net 4))
+  (via (at 111.8 88.265) (size 0.8) (drill 0.4) (layers "F.Cu" "B.Cu") (free) (net 4))
   (via (at 110.395 93.345) (size 0.8) (drill 0.4) (layers "F.Cu" "B.Cu") (net 4))
+  (via (at 121.96 95.885) (size 0.8) (drill 0.4) (layers "F.Cu" "B.Cu") (free) (net 4))
   (via (at 129.445 94.615) (size 0.8) (drill 0.4) (layers "F.Cu" "B.Cu") (net 4))
+  (via (at 134.66 93.345) (size 0.8) (drill 0.4) (layers "F.Cu" "B.Cu") (free) (net 4))
+  (via (at 114.34 90.805) (size 0.8) (drill 0.4) (layers "F.Cu" "B.Cu") (free) (net 4))
+  (via (at 111.8 111.125) (size 0.8) (drill 0.4) (layers "F.Cu" "B.Cu") (free) (net 4))
+  (via (at 127.04 106.045) (size 0.8) (drill 0.4) (layers "F.Cu" "B.Cu") (free) (net 4))
+  (via (at 111.8 103.505) (size 0.8) (drill 0.4) (layers "F.Cu" "B.Cu") (free) (net 4))
+  (via (at 106.72 93.345) (size 0.8) (drill 0.4) (layers "F.Cu" "B.Cu") (free) (net 4))
+  (via (at 127.04 88.265) (size 0.8) (drill 0.4) (layers "F.Cu" "B.Cu") (free) (net 4))
+  (via (at 132.12 90.805) (size 0.8) (drill 0.4) (layers "F.Cu" "B.Cu") (free) (net 4))
+  (via (at 119.42 108.585) (size 0.8) (drill 0.4) (layers "F.Cu" "B.Cu") (free) (net 4))
+  (via (at 127.04 103.505) (size 0.8) (drill 0.4) (layers "F.Cu" "B.Cu") (free) (net 4))
+  (via (at 106.72 95.885) (size 0.8) (drill 0.4) (layers "F.Cu" "B.Cu") (free) (net 4))
   (segment (start 127.225 94.554) (end 127.286 94.615) (width 0.25) (layer "F.Cu") (net 5))
   (segment (start 124.14 101.825) (end 124.14 102.87) (width 0.25) (layer "F.Cu") (net 5))
-  (segment (start 124.46 102.55) (end 124.14 102.87) (width 0.25) (layer "F.Cu") (net 5))
   (segment (start 126.571 100.41) (end 130.81 100.41) (width 0.25) (layer "F.Cu") (net 5))
   (segment (start 127.225 93.0125) (end 127.225 94.554) (width 0.25) (layer "F.Cu") (net 5))
@@
   (segment (start 126.27 100.711) (end 126.571 100.41) (width 0.25) (layer "F.Cu") (net 5))
   (segment (start 124.46 101.505) (end 124.14 101.825) (width 0.25) (layer "F.Cu") (net 5))
-  (segment (start 124.46 100.695) (end 124.745 100.41) (width 0.25) (layer "F.Cu") (net 5))
   (segment (start 124.46 100.695) (end 124.476 100.711) (width 0.25) (layer "F.Cu") (net 5))
   (via (at 127.286 94.615) (size 0.8) (drill 0.4) (layers "F.Cu" "B.Cu") (net 5))
@@
   (segment (start 115.856 93.345) (end 116.6535 92.5475) (width 0.25) (layer "F.Cu") (net 6))
   (segment (start 114.475 98.695) (end 113.98 98.2) (width 0.25) (layer "F.Cu") (net 6))
-  (segment (start 127.54 96.79) (end 127.27 96.52) (width 0.25) (layer "F.Cu") (net 6))
   (segment (start 113.98 98.2) (end 113.98 95.885) (width 0.25) (layer "F.Cu") (net 6))
   (segment (start 113.98 93.345) (end 115.856 93.345) (width 0.25) (layer "F.Cu") (net 6))

Commit message: готово
Changed lines of the file:
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@@
       (psa4output false)
       (plotreference true)
-      (plotvalue true)
+      (plotvalue false)
       (plotinvisibletext false)
       (sketchpadsonfab false)
@@
       (outputformat 1)
       (mirror false)
-      (drillshape 1)
+      (drillshape 0)
       (scaleselection 1)
-      (outputdirectory "")
+      (outputdirectory "../../../kd/")
     )
   )
@@
     (fp_line (start -1 -0.625) (end 1 -0.625) (layer "F.Fab") (width 0.1))
     (fp_line (start 1 0.625) (end -1 0.625) (layer "F.Fab") (width 0.1))
-    (pad "1" smd roundrect (at -1 0 270) (size 1.2 1.4) (layers "F.Cu" "F.Paste" "F.Mask") (roundrect_rratio 0.208333)
+    (pad "1" smd roundrect (at -1 0 270) (size 1.2 1.4) (layers "F.Cu" "F.Paste" "F.Mask") (roundrect_rratio 0.2083333333)
       (net 6 "Net-(C3-Pad1)") (pintype "passive"))
-    (pad "2" smd roundrect (at 1 0 270) (size 1.2 1.4) (layers "F.Cu" "F.Paste" "F.Mask") (roundrect_rratio 0.208333)
+    (pad "2" smd roundrect (at 1 0 270) (size 1.2 1.4) (layers "F.Cu" "F.Paste" "F.Mask") (roundrect_rratio 0.2083333333)
       (net 1 "Net-(C1-Pad1)") (pintype "passive"))
     (model "${KICAD6_3DMODEL_DIR}/Resistor_SMD.3dshapes/R_0805_2012Metric.wrl"
@@
     (fp_line (start -1 -0.625) (end 1 -0.625) (layer "F.Fab") (width 0.1))
     (fp_line (start 1 0.625) (end -1 0.625) (layer "F.Fab") (width 0.1))
-    (pad "1" smd roundrect (at -1 0 180) (size 1.2 1.4) (layers "F.Cu" "F.Paste" "F.Mask") (roundrect_rratio 0.208333)
+    (pad "1" smd roundrect (at -1 0 180) (size 1.2 1.4) (layers "F.Cu" "F.Paste" "F.Mask") (roundrect_rratio 0.2083333333)
       (net 8 "Net-(D1-Pad2)") (pintype "passive"))
-    (pad "2" smd roundrect (at 1 0 180) (size 1.2 1.4) (layers "F.Cu" "F.Paste" "F.Mask") (roundrect_rratio 0.208333)
+    (pad "2" smd roundrect (at 1 0 180) (size 1.2 1.4) (layers "F.Cu" "F.Paste" "F.Mask") (roundrect_rratio 0.2083333333)
       (net 6 "Net-(C3-Pad1)") (pintype "passive"))
     (model "${KICAD6_3DMODEL_DIR}/Resistor_SMD.3dshapes/R_0805_2012Metric.wrl"
@@
     (fp_line (start 1 -0.625) (end 1 0.625) (layer "F.Fab") (width 0.1))
     (fp_line (start 1 0.625) (end -1 0.625) (layer "F.Fab") (width 0.1))
-    (pad "1" smd roundrect (at -1 0 270) (size 1.2 1.4) (layers "F.Cu" "F.Paste" "F.Mask") (roundrect_rratio 0.208333)
+    (pad "1" smd roundrect (at -1 0 270) (size 1.2 1.4) (layers "F.Cu" "F.Paste" "F.Mask") (roundrect_rratio 0.2083333333)
       (net 6 "Net-(C3-Pad1)") (pintype "passive"))
-    (pad "2" smd roundrect (at 1 0 270) (size 1.2 1.4) (layers "F.Cu" "F.Paste" "F.Mask") (roundrect_rratio 0.208333)
+    (pad "2" smd roundrect (at 1 0 270) (size 1.2 1.4) (layers "F.Cu" "F.Paste" "F.Mask") (roundrect_rratio 0.2083333333)
       (net 2 "/out1") (pintype "passive"))
     (model "${KICAD6_3DMODEL_DIR}/Resistor_SMD.3dshapes/R_0805_2012Metric.wrl"
@@
     (fp_line (start -1 0.625) (end -1 -0.625) (layer "F.Fab") (width 0.1))
     (fp_line (start -1 -0.625) (end 1 -0.625) (layer "F.Fab") (width 0.1))
-    (pad "1" smd roundrect (at -1 0 270) (size 1.2 1.4) (layers "F.Cu" "F.Paste" "F.Mask") (roundrect_rratio 0.208333)
+    (pad "1" smd roundrect (at -1 0 270) (size 1.2 1.4) (layers "F.Cu" "F.Paste" "F.Mask") (roundrect_rratio 0.2083333333)
       (net 6 "Net-(C3-Pad1)") (pintype "passive"))
-    (pad "2" smd roundrect (at 1 0 270) (size 1.2 1.4) (layers "F.Cu" "F.Paste" "F.Mask") (roundrect_rratio 0.208333)
+    (pad "2" smd roundrect (at 1 0 270) (size 1.2 1.4) (layers "F.Cu" "F.Paste" "F.Mask") (roundrect_rratio 0.2083333333)
       (net 5 "/out2") (pintype "passive"))
     (model "${KICAD6_3DMODEL_DIR}/Resistor_SMD.3dshapes/R_0805_2012Metric.wrl"
@@
     (fp_line (start 1 -0.625) (end 1 0.625) (layer "F.Fab") (width 0.1))
     (fp_line (start -1 -0.625) (end 1 -0.625) (layer "F.Fab") (width 0.1))
-    (pad "1" smd roundrect (at -1 0 270) (size 1.2 1.4) (layers "F.Cu" "F.Paste" "F.Mask") (roundrect_rratio 0.208333)
+    (pad "1" smd roundrect (at -1 0 270) (size 1.2 1.4) (layers "F.Cu" "F.Paste" "F.Mask") (roundrect_rratio 0.2083333333)
       (net 6 "Net-(C3-Pad1)") (pintype "passive"))
-    (pad "2" smd roundrect (at 1 0 270) (size 1.2 1.4) (layers "F.Cu" "F.Paste" "F.Mask") (roundrect_rratio 0.208333)
+    (pad "2" smd roundrect (at 1 0 270) (size 1.2 1.4) (layers "F.Cu" "F.Paste" "F.Mask") (roundrect_rratio 0.2083333333)
       (net 3 "Net-(C2-Pad2)") (pintype "passive"))
     (model "${KICAD6_3DMODEL_DIR}/Resistor_SMD.3dshapes/R_0805_2012Metric.wrl"
