File: hardware/multivib.kicad_sch (KiCad schematic)
At the start: 20 parts, among them J1 KLS2-301-5.00-02P-2S, J2 KLS2-301-5.00-02P-2S, J3 KLS2-301-5.00-02P-2S, Q1 BC817, Q2 BC817, Q3 2N7002

Commit message: готово
Parts:
- H1, H2, H3, H4: now left out of the parts list
Changed lines of the file:
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@@
   )
   (symbol (lib_id "Mechanical:MountingHole") (at 186.69 128.27 0) (unit 1)
-    (in_bom yes) (on_board yes) (fields_autoplaced)
+    (in_bom no) (on_board yes) (fields_autoplaced)
     (property "Reference" "H2" (id 0) (at 189.23 126.9999 0)
       (effects (font (size 1.27 1.27)) (justify left))
@@
   )
   (symbol (lib_id "Mechanical:MountingHole") (at 186.69 133.35 0) (unit 1)
-    (in_bom yes) (on_board yes) (fields_autoplaced)
+    (in_bom no) (on_board yes) (fields_autoplaced)
     (property "Reference" "H3" (id 0) (at 189.23 132.0799 0)
       (effects (font (size 1.27 1.27)) (justify left))
@@
   )
   (symbol (lib_id "Mechanical:MountingHole") (at 186.69 123.19 0) (unit 1)
-    (in_bom yes) (on_board yes) (fields_autoplaced)
+    (in_bom no) (on_board yes) (fields_autoplaced)
     (property "Reference" "H1" (id 0) (at 189.23 121.9199 0)
       (effects (font (size 1.27 1.27)) (justify left))
@@
   )
   (symbol (lib_id "Mechanical:MountingHole") (at 186.69 138.43 0) (unit 1)
-    (in_bom yes) (on_board yes) (fields_autoplaced)
+    (in_bom no) (on_board yes) (fields_autoplaced)
     (property "Reference" "H4" (id 0) (at 189.23 137.1599 0)
       (effects (font (size 1.27 1.27)) (justify left))
